Commit message: car changed to 4 wheeled car

File: Simulation/racecar.xacro (robot description, xacro)
@@ -1,13 +1,14 @@
 <?xml version="1.0"?>
+<!-- A simple model of the racecar for rviz -->
 <robot xmlns:xacro="http://www.ros.org/wiki/xacro" name="racecar">
-  <xacro:property name="wheelbase" value="1.625" />
-  <xacro:property name="width" value="1.0" />
-  <xacro:property name="height" value="0.5" />
-  <xacro:property name="ground_offset" value="0.2" />
-  <xacro:property name="wheel_radius" value="0.25" />
-  <xacro:property name="wheel_length" value="0.225" />
-  <xacro:property name="laser_distance_from_base_link" value="1.375" />
-  <xacro:property name="laser_height" value="0.25" />
-  <xacro:property name="laser_radius" value="0.13" />
+  <xacro:property name="wheelbase" value="0.325" />
+  <xacro:property name="width" value="0.2" />
+  <xacro:property name="height" value="0.1" />
+  <xacro:property name="ground_offset" value="0.04" />
+  <xacro:property name="wheel_radius" value="0.05" />
+  <xacro:property name="wheel_length" value="0.045" />
+  <xacro:property name="laser_distance_from_base_link" value="0.275" />
+  <xacro:property name="laser_height" value="0.05" />
+  <xacro:property name="laser_radius" value="0.026" />
   <material name="black">
     <color rgba="0.2 0.2 0.2 1."/>
@@ -16,189 +17,105 @@
     <color rgba="0.3 0.57 1. 1."/>
   </material>
-  <material name="dark">
-    <color rgba="0.3 0.3 0.3 1.0"/>
-  </material>
-  <link name="base_footprint"/>
-  <joint name="base_joint" type="fixed">
-    <parent link="base_footprint"/>
-    <child link="base_link" />
-    <origin xyz="0 0 0.1675" rpy="0 0 0.0"/>
-  </joint>
   <link name="base_link">
     <visual>
-      <origin xyz="0.15 -0.325 -0.11" rpy="0 0 1.57"/>
+      <origin xyz="${wheelbase/2} 0 ${ground_offset+height/2}"/>
       <geometry>
-        <mesh filename="package://racecar_simulator/meshes/bases/mini_frame.stl" scale="0.005 0.005 0.005"/>
+        <box size="${wheelbase} ${width} ${height}"/>
       </geometry>
-      <material name="dark"/>
+      <material name="blue"/>
     </visual>
-    <collision>
-      <origin xyz="0.15 -0.325 -0.11" rpy="0 0 1.57"/>
-      <geometry>
-        <mesh filename="package://racecar_simulator/meshes/bases/mini_frame.stl" scale="0.005 0.005 0.005"/>
-      </geometry>
-    </collision>
-    <inertial>
-      <origin xyz="-0.5 0 0" rpy="0 0 0"/>
-      <mass value="6.864548"/>
-      <inertia ixx="0.043501359" ixy="-0.0002378829" ixz="0.00055802495"
-               iyy="0.043097709" iyz="-0.00001771115"
-               izz="0.073063635"/>
-    </inertial>
   </link>
-  <link name="center"/>
+  <link name="center">
+  </link>
   <joint name="base_to_center" type="fixed">
     <parent link="base_link"/>
     <child link="center"/>
-    <origin xyz="0.075 0 0"/>
+    <origin xyz="${wheelbase/2} 0 0"/>
   </joint>
-  <link name="head"/>
+  <link name="head">
+  </link>
   <joint name="base_to_head" type="fixed">
     <parent link="base_link"/>
     <child link="head"/>
-    <origin xyz="0.15 0 0"/>
+    <origin xyz="${wheelbase} 0 0"/>
   </joint>
-  <joint name="housing_joint" type="fixed">
+  <joint name="base_to_laser_model" type="fixed">
     <parent link="base_link"/>
-    <child link="housing_link" />
-    <origin xyz="0 0 0" rpy="0 0 0.0"/>
+    <child link="laser_model"/>
+    <origin xyz="${laser_distance_from_base_link} 0 ${ground_offset+height+(laser_height/2)}"/>
   </joint>
-  <link name="housing_link">
+  <link name="laser_model">
     <visual>
-      <origin xyz="-0.14 0 -0.14" rpy="0 0 1.57"/>
       <geometry>
-        <mesh filename="package://racecar_simulator/meshes/bases/r1mini housing lite 2.stl" scale="0.005 0.005 0.005"/>
+        <cylinder radius="${laser_radius}" length="${laser_height}"/>
       </geometry>
-      <material name="blue"/>
+      <material name="black"/>
     </visual>
-    <collision>
-      <origin xyz="-0.14 0 -0.14" rpy="0 0 1.57"/>
+  </link>
+  <joint name="base_to_back_left_wheel" type="fixed">
+    <parent link="base_link"/>
+    <child link="back_left_wheel"/>
+    <origin xyz="0 ${(wheel_length+width)/2} ${wheel_radius}"/>
+  </joint>
+  <link name="back_left_wheel">
+    <visual>
       <geometry>
-        <mesh filename="package://racecar_simulator/meshes/bases/r1mini housing lite 2.stl" scale="0.005 0.005 0.005"/>
+        <cylinder radius="${wheel_radius}" length="${wheel_length}"/>
       </geometry>
-    </collision>
-    <inertial>
-      <origin xyz="-0.5 0 0" rpy="0 0 0"/>
-      <mass value="0.05"/>
-      <inertia ixx="0.0043501359" ixy="-2.3788291e-06" ixz="5.5802495e-07"
-               iyy="0.0043097709" iyz="-1.771115e-06"
-               izz="0.00073063635"/>
-    </inertial>
+      <material name="black"/>
+      <origin rpy="${pi/2} 0 0"/>
+    </visual>
   </link>
-  <joint name="imu_joint" type="fixed">
+  <joint name="base_to_back_right_wheel" type="fixed">
     <parent link="base_link"/>
-    <child link="imu_link"/>
-    <origin xyz="0.0 0 0.19" rpy="0 0 0"/>
+    <child link="back_right_wheel"/>
+    <origin xyz="0 ${-(wheel_length+width)/2} ${wheel_radius}"/>
   </joint>
-  <link name="imu_link"/>
-  <joint name="scan_joint" type="fixed">
+  <link name="back_right_wheel">
+    <visual>
+      <geometry>
+        <cylinder radius="${wheel_radius}" length="${wheel_length}"/>
+      </geometry>
+      <material name="black"/>
+      <origin rpy="${pi/2} 0 0"/>
+    </visual>
+  </link>
+  <joint name="base_to_front_left_hinge" type="fixed">
     <parent link="base_link"/>
-    <child link="base_scan"/>
-    <origin xyz="0.0 0 0.35" rpy="0.0 0 3.14159"/>
+    <child link="front_left_hinge"/>
+    <origin xyz="${wheelbase} ${(wheel_length+width)/2} ${wheel_radius}"/>
   </joint>
-  <link name="base_scan">
+  <link name="front_left_hinge"/>
+  <joint name="front_left_hinge_to_wheel" type="continuous">
+    <parent link="front_left_hinge"/>
+    <child link="front_left_wheel"/>
+  </joint>
+  <link name="front_left_wheel">
     <visual>
-      <origin xyz="0 0 0.0" rpy="0 0 0"/>
       <geometry>
-        <mesh filename="package://racecar_simulator/meshes/sensors/lds.stl" scale="0.005 0.005 0.005"/>
+        <cylinder radius="${wheel_radius}" length="${wheel_length}"/>
       </geometry>
-      <material name="dark"/>
+      <material name="black"/>
+      <origin rpy="${pi/2} 0 0"/>
     </visual>
-    <collision>
-      <origin xyz="0.075 0 -0.0325" rpy="0 0 0"/>
+  </link>
+  <joint name="base_to_front_right_hinge" type="fixed">
+    <parent link="base_link"/>
+    <child link="front_right_hinge"/>
+    <origin xyz="${wheelbase} ${-(wheel_length+width)/2} ${wheel_radius}"/>
+  </joint>
+  <link name="front_right_hinge"/>
+  <joint name="front_right_hinge_to_wheel" type="continuous">
+    <parent link="front_right_hinge"/>
+    <child link="front_right_wheel"/>
+  </joint>
+  <link name="front_right_wheel">
+    <visual>
       <geometry>
-        <cylinder length="0.1575" radius="0.275"/>
+        <cylinder radius="${wheel_radius}" length="${wheel_length}"/>
       </geometry>
-    </collision>
-    <inertial>
-      <mass value="0.25"/>
-      <origin xyz="0 0 0"/>
-      <inertia ixx="0.005" ixy="0.0" ixz="0.0"
-               iyy="0.005" iyz="0.0"
-               izz="0.005"/>
-    </inertial>
-  </link>
-  <joint name="wheel_left_joint" type="continuous">
-    <parent link="base_link"/>
-    <child link="wheel_left_link"/>
-    <origin xyz="0.0 0.48 0.0" rpy="0.0 0.0 0"/>
-    <axis xyz="0 1 0"/>
-  </joint>
-  <link name="wheel_left_link">
-    <visual>
-      <origin xyz="-0.1675 -0.02 -0.1675" rpy="1.57 0 0"/>
-      <geometry>
-        <mesh filename="package://racecar_simulator/meshes/wheels/mini_tire.stl" scale="0.005 0.005 0.005"/>
-      </geometry>
-      <material name="dark"/>
+      <material name="black"/>
+      <origin rpy="${pi/2} 0 0"/>
     </visual>
-    <collision>
-      <origin xyz="-0.1675 -0.02 -0.1675" rpy="1.57 0 0"/>
-      <geometry>
-        <mesh filename="package://racecar_simulator/meshes/wheels/mini_tire.stl" scale="0.005 0.005 0.005"/>
-      </geometry>
-    </collision>
-    <inertial>
-      <origin xyz="0 0 0"/>
-      <mass value="0.1424947"/>
-      <inertia ixx="0.0000558779" ixy="-2.6429739e-10" ixz="-8.8782569e-08"
-               iyy="0.00005596207" iyz="-7.2000535e-11"
-               izz="0.00010356279"/>
-    </inertial>
-  </link>
-  <joint name="wheel_right_joint" type="continuous">
-    <parent link="base_link"/>
-    <child link="wheel_right_link"/>
-    <origin xyz="0.0 -0.48 0.0" rpy="0.0 0.0 0"/>
-    <axis xyz="0 1 0"/>
-  </joint>
-  <link name="wheel_right_link">
-    <visual>
-      <origin xyz="-0.1675 0.02 0.1675" rpy="-1.57 0 0"/>
-      <geometry>
-        <mesh filename="package://racecar_simulator/meshes/wheels/mini_tire.stl" scale="0.005 0.005 0.005"/>
-      </geometry>
-      <material name="dark"/>
-    </visual>
-    <collision>
-      <origin xyz="-0.1675 0.02 0.1675" rpy="-1.57 0 0"/>
-      <geometry>
-        <mesh filename="package://racecar_simulator/meshes/wheels/mini_tire.stl" scale="0.005 0.005 0.005"/>
-      </geometry>
-    </collision>
-    <inertial>
-      <origin xyz="0 0 0"/>
-      <mass value="0.1424947"/>
-      <inertia ixx="0.0000558779" ixy="-2.6429739e-10" ixz="-8.8782569e-08"
-               iyy="0.00005596207" iyz="-7.2000535e-11"
-               izz="0.00010356279"/>
-    </inertial>
-  </link>
-  <joint name="caster_back_joint" type="fixed">
-    <parent link="base_link"/>
-    <child link="caster_back_link"/>
-    <origin xyz="-0.6 0.0 -0.09" rpy="0 0 0"/>
-  </joint>
-  <link name="caster_back_link">
-    <visual>
-      <origin xyz="-0.08 -0.035 -0.08" rpy="0 0 0"/>
-      <geometry>
-        <mesh filename="package://racecar_simulator/meshes/wheels/mini_caster.stl" scale="0.005 0.005 0.005"/>
-      </geometry>
-      <material name="dark"/>
-    </visual>
-    <collision>
-      <origin xyz="-0.08 -0.035 -0.08" rpy="0 0 0"/>
-      <geometry>
-        <mesh filename="package://racecar_simulator/meshes/wheels/mini_caster.stl" scale="0.005 0.005 0.005"/>
-      </geometry>
-    </collision>
-    <inertial>
-      <origin xyz="0 0 0"/>
-      <mass value="0.025"/>
-      <inertia ixx="0.005" ixy="0.0" ixz="0.0"
-               iyy="0.005" iyz="0.0"
-               izz="0.005"/>
-    </inertial>
   </link>
 </robot>
